File: SeniorDesignProject/SeniorDesign.sch (KiCad schematic (older format))
At the start: 44 parts, among them J1 RJ45, P1 CONN_01X03, P2 CONN_01X03, P3 CONN_01X03, P4 CONN_01X03, P5 CONN_01X06, P6 CONN_01X05, P7 CONN_01X02, P8 CONN_01X05, U1 LM741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

Commit message: updates
Parts:
- removed C2, C3, C4, C5, C6, C7, C8: 100nF, Capacitors_SMD:C_0201, symbol C
- removed R10, R2, R3, R5, R9: 47, Resistors_SMD:R_0805, symbol R
- removed R11, R12: 3300, Resistors_SMD:R_0805, symbol R
- removed R4, R6, R7, R8: 2700, Resistors_SMD:R_0805, symbol R
- removed U1, U2, U3, U4, U5, U6, U7, U8: LM741, Housings_DIP:DIP-8_W7.62mm, symbol LM741-RESCUE-SeniorDesign
- removed U11: LM2931Z-3.3/5.0, TO_SOT_Packages_THT:TO-220_Neutral123_Vertical, symbol LM2931Z-3.3/5.0
- added J2: RJ45, Connect:RJ45_8, symbol RJ45
- added LC2, LC3, LC4: a14071900ux0061, SeniorDesignFootprints:a14071900ux0061, symbol a14071900ux0061
- added U1: INA827, Housings_SSOP:MSOP-8_3x3mm_Pitch0.65mm, symbol INA827
- C1: value 100nF -> C; footprint Capacitors_SMD:C_0201 -> Capacitors_SMD:C_0805
- LC1: footprint (none) -> SeniorDesignFootprints:a14071900ux0061
- P1, P2, P3, P4: footprint Pin_Headers:Pin_Header_Angled_1x03 -> Pin_Headers:Pin_Header_Angled_1x03_Pitch2.54mm
- P5: footprint Pin_Headers:Pin_Header_Straight_1x06 -> Pin_Headers:Pin_Header_Straight_1x06_Pitch2.54mm
- P6: footprint Pin_Headers:Pin_Header_Straight_1x05 -> Pin_Headers:Pin_Header_Straight_1x05_Pitch2.54mm
- R1: value 47 -> 80.6
Connections:
- net labels removed: +5V, Earth
- wire segments 82 -> 4
Other:
- moved on the sheet: J1, P7

Commit message: updates 1/30/2017
Parts:
- removed XB1: XBee-SX, SeniorDesignFootprints:XBEE_SX, symbol XBee-SX
- added P9: XBEE-Headers, _connectors1:XBEE-HEADER, symbol XBEE-Headers
Changed lines of the file:
@@
-$EndComp
-$Comp
-L XBee-SX XB1
-U 1 1 5845B1A4
-P 5415 6565
-F 0 "XB1" H 5415 7365 60  0000 C CNN
-F 1 "XBee-SX" H 5390 7490 98  0000 C CNN
-F 2 "SeniorDesignFootprints:XBEE_SX" H 3940 5740 60  0001 C CNN
-F 3 "" H 3940 5740 60  0001 C CNN
-	1    5415 6565
-	1    0    0    -1
 $EndComp
 $Comp
@@
 L CONN_01X03 P3
 U 1 1 584603A4
-P 770 5090
-F 0 "P3" H 770 5290 50  0000 C CNN
-F 1 "CONN_01X03" V 870 5090 50  0000 C CNN
-F 2 "Pin_Headers:Pin_Header_Angled_1x03_Pitch2.54mm" H 770 5090 50  0001 C CNN
-F 3 "" H 770 5090 50  0000 C CNN
-	1    770  5090
+P 825 5090
+F 0 "P3" H 825 5290 50  0000 C CNN
+F 1 "CONN_01X03" V 925 5090 50  0000 C CNN
+F 2 "Pin_Headers:Pin_Header_Angled_1x03_Pitch2.54mm" H 825 5090 50  0001 C CNN
+F 3 "" H 825 5090 50  0000 C CNN
+	1    825  5090
 	1    0    0    -1
 $EndComp
@@
 	1    0    0    -1
 $EndComp
+$Comp
+L XBEE-Headers P9
+U 1 1 588F841D
+P 3515 4410
+F 0 "P9" H 3215 5060 50  0000 C CNN
+F 1 "XBEE-Headers" H 3215 4960 50  0000 C CNN
+F 2 "_connectors1:XBEE-HEADER" H 3415 4410 50  0001 C CNN
+F 3 "" H 3415 4410 50  0001 C CNN
+	1    3515 4410
+	1    0    0    -1
+$EndComp

Commit message: Updates to the project
Parts:
- removed C1: C, Capacitors_SMD:C_0805, symbol C
- removed LC1, LC2, LC3, LC4: a14071900ux0061, SeniorDesignFootprints:a14071900ux0061, symbol a14071900ux0061
- removed P9: XBEE-Headers, _connectors1:XBEE-HEADER, symbol XBEE-Headers
- added C? (x5): 0.1uF, symbol C
- added C?: 4.7uF, symbol C
- added C? (x2): C, symbol C
- added P?: CONN_01X02, Pin_Headers:Pin_Header_Straight_1x02_Pitch3.96mm_Friction_Lock, symbol CONN_01X02
- added R?: 10k, symbol R
Connections:
- net labels added: +5V, -5V, 3.3V, GND
- wire segments 4 -> 45
Other:
- moved on the sheet: CPU1, P7, R1, U1, U10, U9

Commit message: Updates to board
Parts:
- removed P1, P2, P3, P4: CONN_01X03, Pin_Headers:Pin_Header_Angled_1x03_Pitch2.54mm, symbol CONN_01X03
- removed P5: CONN_01X06, Pin_Headers:Pin_Header_Straight_1x06_Pitch2.54mm, symbol CONN_01X06
- removed P6: CONN_01X05, Pin_Headers:Pin_Header_Straight_1x05_Pitch2.54mm, symbol CONN_01X05
- removed P8: CONN_01X05, Socket_Strips:Socket_Strip_Straight_1x05, symbol CONN_01X05
- removed RF1: ID-12LA, SeniorDesignFootprints:ID-12LA, symbol ID-12LA
- added J3: PICkit3, Pin_Headers:Pin_Header_Straight_1x06_Pitch2.54mm, symbol CONN_01X06
- added J4: RJ11(ICD3), SeniorDesignFootprints:RJ11-6, symbol RJ11
- added J5: ID-12LA Header, Pin_Headers:Pin_Header_Straight_2x06_Pitch2.54mm, symbol CONN_02X06
- added J6: XBEE Header, SeniorDesignFootprints:XBEE-HEADER, symbol CONN_02X10
- C1, C2: renamed from C?; value C -> 0.1uF; footprint (none) -> Capacitors_SMD:C_0805
- C3, C4, C5, C6, C7: renamed from C?; footprint (none) -> Capacitors_SMD:C_0805
- C8: renamed from C?; footprint (none) -> Capacitors_SMD:CP_Elec_4x4.5
- J1: value RJ45 -> RJ45(LoadCells)
- J2: value RJ45 -> RJ45(Accelerometer)
- P7: value CONN_01X02 -> Power 1
- P9: renamed from P?; value CONN_01X02 -> Power 2
- R2: renamed from R?; footprint (none) -> Resistors_SMD:R_0805
Connections:
- wire segments 45 -> 38
Other:
- moved on the sheet: P9
Changed lines of the file:
@@
-$EndComp
-$Comp
-L ID-12LA RF1
-U 1 1 5845DD1D
-P 2330 6660
-F 0 "RF1" H 2305 6985 60  0000 C CNN
-F 1 "ID-12LA" H 2305 7110 98  0000 C CNN
-F 2 "SeniorDesignFootprints:ID-12LA" H 1730 4535 60  0001 C CNN
-F 3 "https://cdn.sparkfun.com/datasheets/Sensors/ID/ID-2LA,%20ID-12LA,%20ID-20LA2013-4-10.pdf" H 1730 4535 60  0001 C CNN
-	1    2330 6660
-	1    0    0    -1
 $EndComp
 $Comp
@@
 P 720 795
 F 0 "P7" H 720 945 50  0000 C CNN
-F 1 "CONN_01X02" V 820 795 50  0000 C CNN
+F 1 "Power 1" V 820 795 50  0000 C CNN
 F 2 "Pin_Headers:Pin_Header_Straight_1x02_Pitch3.96mm_Friction_Lock" H 720 795 50  0001 C CNN
 F 3 "" H 720 795 50  0000 C CNN
 	1    720  795
 	-1   0    0    1
-$EndComp
-$Comp
-L CONN_01X03 P3
-U 1 1 584603A4
-P 825 5090
-F 0 "P3" H 825 5290 50  0000 C CNN
-F 1 "CONN_01X03" V 925 5090 50  0000 C CNN
-F 2 "Pin_Headers:Pin_Header_Angled_1x03_Pitch2.54mm" H 825 5090 50  0001 C CNN
-F 3 "" H 825 5090 50  0000 C CNN
-	1    825  5090
-	1    0    0    -1
-$EndComp
-$Comp
-L CONN_01X03 P1
-U 1 1 58460427
-P 815 6820
-F 0 "P1" H 815 7020 50  0000 C CNN
-F 1 "CONN_01X03" V 915 6820 50  0000 C CNN
-F 2 "Pin_Headers:Pin_Header_Angled_1x03_Pitch2.54mm" H 815 6820 50  0001 C CNN
-F 3 "" H 815 6820 50  0000 C CNN
-	1    815  6820
-	1    0    0    -1
-$EndComp
-$Comp
-L CONN_01X03 P2
-U 1 1 584604A0
-P 805 5665
-F 0 "P2" H 805 5865 50  0000 C CNN
-F 1 "CONN_01X03" V 905 5665 50  0000 C CNN
-F 2 "Pin_Headers:Pin_Header_Angled_1x03_Pitch2.54mm" H 805 5665 50  0001 C CNN
-F 3 "" H 805 5665 50  0000 C CNN
-	1    805  5665
-	1    0    0    -1
-$EndComp
-$Comp
-L CONN_01X03 P4
-U 1 1 584605AB
-P 830 6250
-F 0 "P4" H 830 6450 50  0000 C CNN
-F 1 "CONN_01X03" V 930 6250 50  0000 C CNN
-F 2 "Pin_Headers:Pin_Header_Angled_1x03_Pitch2.54mm" H 830 6250 50  0001 C CNN
-F 3 "" H 830 6250 50  0000 C CNN
-	1    830  6250
-	1    0    0    -1
-$EndComp
-$Comp
-L CONN_01X05 P6
-U 1 1 58460650
-P 5665 1215
-F 0 "P6" H 5665 1515 50  0000 C CNN
-F 1 "CONN_01X05" V 5765 1215 50  0000 C CNN
-F 2 "Pin_Headers:Pin_Header_Straight_1x05_Pitch2.54mm" H 5665 1215 50  0001 C CNN
-F 3 "" H 5665 1215 50  0000 C CNN
-	1    5665 1215
-	1    0    0    -1
-$EndComp
-$Comp
-L CONN_01X05 P8
-U 1 1 584606F1
-P 8805 885
-F 0 "P8" H 8805 1185 50  0000 C CNN
-F 1 "CONN_01X05" V 8905 885 50  0000 C CNN
-F 2 "Socket_Strips:Socket_Strip_Straight_1x05" H 8805 885 50  0001 C CNN
-F 3 "" H 8805 885 50  0000 C CNN
-	1    8805 885
-	1    0    0    -1
-$EndComp
-$Comp
-L CONN_01X06 P5
-U 1 1 58460780
-P 4980 1230
-F 0 "P5" H 4980 1580 50  0000 C CNN
-F 1 "CONN_01X06" V 5080 1230 50  0000 C CNN
-F 2 "Pin_Headers:Pin_Header_Straight_1x06_Pitch2.54mm" H 4980 1230 50  0001 C CNN
-F 3 "" H 4980 1230 50  0000 C CNN
-	1    4980 1230
-	1    0    0    -1
 $EndComp
 $Comp
@@
 U 1 1 584637CE
 P 1130 2250
-F 0 "J1" H 1330 2750 50  0000 C CNN
-F 1 "RJ45" H 980 2750 50  0000 C CNN
+F 0 "J1" H 1590 2255 50  0000 C CNN
+F 1 "RJ45(LoadCells)" H 1130 2770 50  0000 C CNN
 F 2 "Connect:RJ45_8" H 1130 2250 50  0001 C CNN
 F 3 "" H 1130 2250 50  0000 C CNN
@@
 U 1 1 588D56E2
 P 1165 3405
-F 0 "J2" H 1365 3905 50  0000 C CNN
-F 1 "RJ45" H 1015 3905 50  0000 C CNN
+F 0 "J2" H 1650 3410 50  0000 C CNN
+F 1 "RJ45(Accelerometer)" H 1175 3915 50  0000 C CNN
 F 2 "Connect:RJ45_8" H 1165 3405 50  0001 C CNN
 F 3 "" H 1165 3405 50  0000 C CNN
@@
 $EndComp
 $Comp
-L C C?
+L C C4
 U 1 1 58AC7C8B
 P 5275 2890
-F 0 "C?" H 5300 2990 50  0000 L CNN
+F 0 "C4" H 5300 2990 50  0000 L CNN
 F 1 "0.1uF" H 5300 2790 50  0000 L CNN
-F 2 "" H 5313 2740 50  0001 C CNN
+F 2 "Capacitors_SMD:C_0805" H 5313 2740 50  0001 C CNN
 F 3 "" H 5275 2890 50  0001 C CNN
 	1    5275 2890
@@
 $EndComp
 Wire Wire Line
-	4870 2715 5275 2715
-Wire Wire Line
-	5275 2715 5425 2715
+	4870 2715 5425 2715
 Wire Wire Line
 	5450 3040 5450 2930
@@
 	5450 2930 5580 2930
 Wire Wire Line
-	4875 3040 5275 3040
-Wire Wire Line
-	5275 3040 5450 3040
+	4875 3040 5450 3040
 Wire Wire Line
 	5425 2715 5425 2830
@@
 	5425 2830 5580 2830
 $Comp
-L C C?
+L C C5
 U 1 1 58AC8F63
 P 5275 3890
-F 0 "C?" H 5300 3990 50  0000 L CNN
+F 0 "C5" H 5300 3990 50  0000 L CNN
 F 1 "0.1uF" H 5300 3790 50  0000 L CNN
-F 2 "" H 5313 3740 50  0001 C CNN
+F 2 "Capacitors_SMD:C_0805" H 5313 3740 50  0001 C CNN
 F 3 "" H 5275 3890 50  0001 C CNN
 	1    5275 3890
@@
 $EndComp
 Wire Wire Line
-	4870 3720 5275 3720
-Wire Wire Line
-	5275 3720 5425 3720
+	4870 3720 5425 3720
 Wire Wire Line
 	5450 4040 5450 3930
@@
 	5450 3930 5580 3930
 Wire Wire Line
-	4855 4040 5275 4040
-Wire Wire Line
-	5275 4040 5450 4040
+	4855 4040 5450 4040
 Wire Wire Line
 	5425 3720 5425 3830
@@
 	5425 3830 5580 3830
 $Comp
-L C C?
+L C C3
 U 1 1 58AC90D5
 P 5200 4490
-F 0 "C?" H 5225 4590 50  0000 L CNN
+F 0 "C3" H 5225 4590 50  0000 L CNN
 F 1 "0.1uF" H 5225 4390 50  0000 L CNN
-F 2 "" H 5238 4340 50  0001 C CNN
+F 2 "Capacitors_SMD:C_0805" H 5238 4340 50  0001 C CNN
 F 3 "" H 5200 4490 50  0001 C CNN
 	1    5200 4490
@@
 $EndComp
 Wire Wire Line
-	4870 4340 5200 4340
-Wire Wire Line
-	5200 4340 5425 4340
+	4870 4340 5425 4340
 Wire Wire Line
 	5450 4640 5450 4530
@@
 	5450 4530 5580 4530
 Wire Wire Line
-	4870 4640 5200 4640
-Wire Wire Line
-	5200 4640 5450 4640
+	4870 4640 5450 4640
 Wire Wire Line
 	5425 4340 5425 4430
@@
 	5425 4430 5580 4430
 $Comp
-L C C?
+L C C7
 U 1 1 58AC96B7
 P 9910 2360
-F 0 "C?" V 9695 2325 50  0000 L CNN
+F 0 "C7" V 9695 2325 50  0000 L CNN
 F 1 "0.1uF" V 9770 2285 50  0000 L CNN
-F 2 "" H 9948 2210 50  0001 C CNN
+F 2 "Capacitors_SMD:C_0805" H 9948 2210 50  0001 C CNN
 F 3 "" H 9910 2360 50  0001 C CNN
 	1    9910 2360
@@
 	9760 2705 9605 2730
 $Comp
-L C C?
+L C C8
 U 1 1 58ACA467
 P 9915 2880
-F 0 "C?" V 10045 2850 50  0000 L CNN
+F 0 "C8" V 10045 2850 50  0000 L CNN
 F 1 "4.7uF" V 10125 2820 50  0000 L CNN
-F 2 "" H 9953 2730 50  0001 C CNN
+F 2 "Capacitors_SMD:CP_Elec_4x4.5" H 9953 2730 50  0001 C CNN
 F 3 "" H 9915 2880 50  0001 C CNN
 	1    9915 2880
@@
 Connection ~ 5275 2715
 Wire Wire Line
-	9605 4330 9810 4330
-Wire Wire Line
-	9810 4330 10010 4330
-$Comp
-L C C?
+	9605 4330 10010 4330
+$Comp
+L C C6
 U 1 1 58ACD271
 P 9810 4480
-F 0 "C?" H 9830 4405 50  0000 L CNN
+F 0 "C6" H 9830 4405 50  0000 L CNN
 F 1 "0.1uF" H 9835 4575 50  0000 L CNN
-F 2 "" H 9848 4330 50  0001 C CNN
+F 2 "Capacitors_SMD:C_0805" H 9848 4330 50  0001 C CNN
 F 3 "" H 9810 4480 50  0001 C CNN
 	1    9810 4480
@@
 $EndComp
 Wire Wire Line
-	9605 4630 9810 4630
-Wire Wire Line
-	9810 4630 10105 4630
+	9605 4630 10105 4630
 Connection ~ 9810 4330
 Connection ~ 9810 4630
 $Comp
-L R R?
+L R R2
 U 1 1 58ACE239
 P 5200 2500
-F 0 "R?" V 5280 2500 50  0000 C CNN
+F 0 "R2" V 5280 2500 50  0000 C CNN
 F 1 "10k" V 5200 2500 50  0000 C CNN
-F 2 "" V 5130 2500 50  0001 C CNN
+F 2 "Resistors_SMD:R_0805" V 5130 2500 50  0001 C CNN
 F 3 "" H 5200 2500 50  0001 C CNN
 	1    5200 2500
@@
 	3585 3480 3465 3470
 $Comp
-L C C?
+L C C2
 U 1 1 58AD1F47
 P 4035 3025
-F 0 "C?" H 4060 3125 50  0000 L CNN
-F 1 "C" H 4060 2925 50  0000 L CNN
-F 2 "" H 4073 2875 50  0001 C CNN
+F 0 "C2" H 4060 3125 50  0000 L CNN
+F 1 "0.1uF" H 4060 2925 50  0000 L CNN
+F 2 "Capacitors_SMD:C_0805" H 4073 2875 50  0001 C CNN
 F 3 "" H 4035 3025 50  0001 C CNN
 	1    4035 3025
@@
 GND
 Wire Wire Line
-	3885 2870 3885 2915
-Wire Wire Line
-	3885 2915 3885 3025
+	3885 2870 3885 3025
 Connection ~ 3885 2915
 Text GLabel 3585 3680 3    60   Input ~ 0
 GND
 $Comp
-L C C?
+L C C1
 U 1 1 58AD24D1
 P 3735 3680
-F 0 "C?" H 3760 3780 50  0000 L CNN
-F 1 "C" H 3760 3580 50  0000 L CNN
-F 2 "" H 3773 3530 50  0001 C CNN
+F 0 "C1" H 3760 3780 50  0000 L CNN
+F 1 "0.1uF" H 3760 3580 50  0000 L CNN
+F 2 "Capacitors_SMD:C_0805" H 3773 3530 50  0001 C CNN
 F 3 "" H 3735 3680 50  0001 C CNN
 	1    3735 3680
@@
 $EndComp
 Wire Wire Line
-	3885 3620 3885 3675
-Wire Wire Line
-	3885 3675 3885 3680
-$Comp
-L CONN_01X02 P?
+	3885 3620 3885 3680
+$Comp
+L CONN_01X02 P9
 U 1 1 58AD41C9
-P 2385 850
-F 0 "P?" H 2385 1000 50  0000 C CNN
-F 1 "CONN_01X02" V 2485 850 50  0000 C CNN
-F 2 "Pin_Headers:Pin_Header_Straight_1x02_Pitch3.96mm_Friction_Lock" H 2385 850 50  0001 C CNN
-F 3 "" H 2385 850 50  0000 C CNN
-	1    2385 850
-	-1   0    0    1
-$EndComp
+P 730 1360
+F 0 "P9" H 730 1510 50  0000 C CNN
+F 1 "Power 2" V 830 1360 50  0000 C CNN
+F 2 "Pin_Headers:Pin_Header_Straight_1x02_Pitch3.96mm_Friction_Lock" H 730 1360 50  0001 C CNN
+F 3 "" H 730 1360 50  0000 C CNN
+	1    730  1360
+	-1   0    0    1
+$EndComp
+$Comp
+L CONN_02X10 J6
+U 1 1 58ACD0F4
+P 3195 5295
+F 0 "J6" H 3195 5845 50  0000 C CNN
+F 1 "XBEE Header" V 3195 5295 50  0000 C CNN
+F 2 "SeniorDesignFootprints:XBEE-HEADER" H 3195 4095 50  0001 C CNN
+F 3 "" H 3195 4095 50  0001 C CNN
+	1    3195 5295
+	1    0    0    -1
+$EndComp
+$Comp
+L CONN_02X06 J5
+U 1 1 58ACD24B
+P 2390 5270
+F 0 "J5" H 2390 5620 50  0000 C CNN
+F 1 "ID-12LA Header" V 2390 5250 39  0000 C CNN
+F 2 "Pin_Headers:Pin_Header_Straight_2x06_Pitch2.54mm" H 2390 4070 50  0001 C CNN
+F 3 "" H 2390 4070 50  0001 C CNN
+	1    2390 5270
+	1    0    0    -1
+$EndComp
+$Comp
+L RJ11 J4
+U 1 1 58ACD97B
+P 1140 4485
+F 0 "J4" H 1340 4985 60  0000 C CNN
+F 1 "RJ11(ICD3)" H 990 4985 60  0000 C CNN
+F 2 "SeniorDesignFootprints:RJ11-6" H 1140 4485 60  0001 C CNN
+F 3 "" H 1140 4485 60  0001 C CNN
+	1    1140 4485
+	0    -1   -1   0
+$EndComp
+$Comp
+L CONN_01X06 J3
+U 1 1 58ACED75
+P 815 5380
+F 0 "J3" H 815 5730 50  0000 C CNN
+F 1 "PICkit3" V 915 5380 50  0000 C CNN
+F 2 "Pin_Headers:Pin_Header_Straight_1x06_Pitch2.54mm" H 815 5380 50  0001 C CNN
+F 3 "" H 815 5380 50  0001 C CNN
+	1    815  5380
+	-1   0    0    -1
+$EndComp
+Wire Wire Line
+	4285 3320 5425 3320
+Wire Wire Line
+	5425 3320 5425 3230
+Wire Wire Line
+	5425 3230 5580 3230
 $EndSCHEMATC

Commit message: Updates
Parts:
- added J7: 7-Segment Display, Socket_Strips:Socket_Strip_Straight_1x05_Pitch2.54mm, symbol CONN_01X05
- added R3, R4, R5, R6: 4.7k, Resistors_SMD:R_0805, symbol R
- U10, U9: footprint TO_SOT_Packages_THT:TO-220_Neutral123_Vertical -> TO_SOT_Packages_THT:TO-220_Horizontal
Connections:
- net +5V: now also J1.8, J5.1 (P1)
- net 3.3V: now also J2.8, J3.2 (P2), J4.2, J6.1 (P1), J7.1 (P1), R3.2, R4.1, R5.1, R6.1
- net GND: now also J1.7, J2.7, J3.3 (P3), J4.3, J5.4 (P4), J5.9 (P9), J6.10 (P10)
- net AN0: now reaches CPU1.13 (AN0/OA2OUT/RA0), U1.7 (Vout)
- net PGED3: now reaches CPU1.15 (PGED3/VREF-/AN2/C2IN1-/~SS1~/RPI32/CTED2/RB0)
- net PGED3: now also J3.4 (P4), J4.4
- net PGEC3: now reaches CPU1.16 (PGEC3/VREF+/AN3/OA1OUT/RPI33/CTED1/RB1)
- net PGEC3: now also J3.5 (P5), J4.5
- net SDA2: now reaches CPU1.31 (SDA2/RPI24/RA8)
- net SDA2: now also J2.4, R4.2
- net SCL2: now reaches CPU1.32 (FLT32/SCL2/RP36/RB4)
- net SCL2: now also J2.5, R3.1
- net SDA1: now reaches CPU1.36 (SDA1/RPI52/RC4)
- net SDA1: now also J7.4 (P4), R6.2
- net SCL1: now reaches CPU1.37 (SCL1/RPI53/RC5)
- net SCL1: now also J7.5 (P5), R5.2
- net UART1TX: now reaches CPU1.50 (RP54/RC6)
- net UART1RX: now reaches CPU1.51 (RP55/RC7)
- net UART1RX: now also J5.5 (P5)
- net UART2TX: now reaches CPU1.61 (RP43/PWM3L/RB11)
- net UART2TX: now also J6.3 (P3)
- net UART2RX: now reaches CPU1.62 (RPI44/PWM2H/RB12)
- net UART2RX: now also J6.2 (P2)
- net A-: now reaches J1.4
- net A-: now also U1.1 (-)
- net A+: now reaches J1.5
- net A+: now also U1.4 (+)
- net RFID_LED: now reaches J5.3 (P3)
- net MCLR: now reaches J4.1
- net MCLR: now also J3.1 (P1)
- new net +5V(2): J7.2 (P2)
- new net GND(2): J7.3 (P3)
- no-connect marks 0 -> 32
Other:
- moved on the sheet: C1, C2, C3, C4, C5, C6, C7, C8, CPU1, J1, J2, J4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

Commit message: added some traces
Connections:
- net +5V: now also U1.8 (V+)
- net AN0: now also CPU1.28 (AN13/C3IN2-/~U2CTS~/RE13); no longer CPU1.13 (AN0/OA2OUT/RA0)
- net GND: no longer C2.2
- net SCL1: now also CPU1.48 (TCK/CVREF1O/ASCL1/RP40/T4CK/RB8); no longer CPU1.37 (SCL1/RPI53/RC5)
- net SCL2: now also CPU1.44 (PGEC2/ASCL2/RP38/RB6); no longer CPU1.32 (FLT32/SCL2/RP36/RB4)
- net SDA1: now also CPU1.49 (TMS/ASDA1/RP41/RB9); no longer CPU1.36 (SDA1/RPI52/RC4)
- net SDA2: now also CPU1.43 (PGED2/ASDA2/RP37/RB5); no longer CPU1.31 (SDA2/RPI24/RA8)
- net UART1RX: now also CPU1.45 (RPI58/RC10); no longer CPU1.51 (RP55/RC7)
- net UART1TX: now also CPU1.46 (RP39/INT0/RB7); no longer CPU1.50 (RP54/RC6)
Other:
- moved on the sheet: R3, R4, R5, R6
Changed lines of the file:
@@
 L C C2
 U 1 1 58AD1F47
-P 1655 2685
-F 0 "C2" H 1680 2785 50  0000 L CNN
-F 1 "0.1uF" H 1680 2585 50  0000 L CNN
-F 2 "Capacitors_SMD:C_0805" H 1693 2535 50  0001 C CNN
-F 3 "" H 1655 2685 50  0001 C CNN
-	1    1655 2685
+P 1655 2680
+F 0 "C2" V 1855 2640 50  0000 L CNN
+F 1 "0.1uF" V 1775 2580 50  0000 L CNN
+F 2 "Capacitors_SMD:C_0805" H 1693 2530 50  0001 C CNN
+F 3 "" H 1655 2680 50  0001 C CNN
+	1    1655 2680
 	0    -1   -1   0
 $EndComp
@@
 U 1 1 58AD24D1
 P 1355 3340
-F 0 "C1" H 1380 3440 50  0000 L CNN
-F 1 "0.1uF" H 1380 3240 50  0000 L CNN
+F 0 "C1" V 1220 3295 50  0000 L CNN
+F 1 "0.1uF" V 1155 3245 50  0000 L CNN
 F 2 "Capacitors_SMD:C_0805" H 1393 3190 50  0001 C CNN
 F 3 "" H 1355 3340 50  0001 C CNN
@@
 	10105 1570 10105 1560
 Wire Wire Line
-	1505 2530 1505 2685
-Connection ~ 1505 2575
+	1505 2530 1505 2680
+Connection ~ 1505 2570
 Wire Wire Line
 	1505 3280 1505 3340
-$Comp
-L INA827 U1
-U 1 1 588D6159
-P 1505 2980
-F 0 "U1" H 1655 3105 50  0000 L CNN
-F 1 "INA827" H 1655 2855 50  0000 L CNN
-F 2 "Housings_SSOP:MSOP-8_3x3mm_Pitch0.65mm" H 1655 2780 50  0001 L CNN
-F 3 "http://www.ti.com/lit/ds/symlink/ina827.pdf" H 1605 2980 50  0001 C CNN
-	1    1505 2980
-	1    0    0    -1
-$EndComp
 Wire Wire Line
 	935  3130 1205 3080
@@
 NoConn ~ 5570 6690
 NoConn ~ 5670 6690
-Text GLabel 4390 3995 0    39   Input ~ 0
+Text GLabel 10915 2895 2    39   Input ~ 0
 SCL2
-Text GLabel 4725 3895 0    39   Input ~ 0
+Text GLabel 10580 2995 2    39   Input ~ 0
 SDA2
 Text GLabel 5640 2295 0    39   Input ~ 0
@@
 Text GLabel 1030 6420 2    39   Input ~ 0
 SCL1
-Text GLabel 10510 3595 2    39   Input ~ 0
+Text GLabel 10555 2495 2    39   Input ~ 0
 SCL1
-Text GLabel 10880 3695 2    39   Input ~ 0
+Text GLabel 10240 2395 2    39   Input ~ 0
 SDA1
-Text GLabel 5640 2095 0    39   Input ~ 0
+Text GLabel 5640 3595 0    39   Input ~ 0
 AN0
 Text GLabel 1905 2980 2    39   Input ~ 0
@@
 Text GLabel 9665 1095 2    39   Input ~ 0
 UART2RX
-Text GLabel 9665 2195 2    39   Input ~ 0
+Text GLabel 9665 2795 2    39   Input ~ 0
 UART1RX
-Text GLabel 9665 2295 2    39   Input ~ 0
+Text GLabel 9665 2695 2    39   Input ~ 0
 UART1TX
 Wire Wire Line
-	9665 3595 10510 3595
+	9665 2495 10555 2495
 $Comp
 L R R5
 U 1 1 58AE9BED
-P 10465 3445
-F 0 "R5" V 10545 3445 50  0000 C CNN
-F 1 "4.7k" V 10465 3445 50  0000 C CNN
-F 2 "Resistors_SMD:R_0805" V 10395 3445 50  0001 C CNN
-F 3 "" H 10465 3445 50  0001 C CNN
-	1    10465 3445
-	1    0    0    -1
-$EndComp
-Text GLabel 10465 3295 1    39   Input ~ 0
-3.3V
-Connection ~ 10465 3595
-Wire Wire Line
-	9665 3695 10880 3695
+P 10525 2345
+F 0 "R5" V 10605 2345 50  0000 C CNN
+F 1 "4.7k" V 10525 2345 50  0000 C CNN
+F 2 "Resistors_SMD:R_0805" V 10455 2345 50  0001 C CNN
+F 3 "" H 10525 2345 50  0001 C CNN
+	1    10525 2345
+	1    0    0    -1
+$EndComp
+Text GLabel 10525 2195 1    39   Input ~ 0
+3.3V
+Connection ~ 10525 2495
+Wire Wire Line
+	9665 2395 10240 2395
 $Comp
 L R R6
 U 1 1 58AEA269
-P 10830 3545
-F 0 "R6" V 10910 3545 50  0000 C CNN
-F 1 "4.7k" V 10830 3545 50  0000 C CNN
-F 2 "Resistors_SMD:R_0805" V 10760 3545 50  0001 C CNN
-F 3 "" H 10830 3545 50  0001 C CNN
-	1    10830 3545
-	1    0    0    -1
-$EndComp
-Text GLabel 10830 3395 1    39   Input ~ 0
-3.3V
-Connection ~ 10830 3695
-Wire Wire Line
-	4725 3895 5640 3895
+P 10190 2245
+F 0 "R6" V 10270 2245 50  0000 C CNN
+F 1 "4.7k" V 10190 2245 50  0000 C CNN
+F 2 "Resistors_SMD:R_0805" V 10120 2245 50  0001 C CNN
+F 3 "" H 10190 2245 50  0001 C CNN
+	1    10190 2245
+	1    0    0    -1
+$EndComp
+Text GLabel 10190 2095 1    39   Input ~ 0
+3.3V
+Connection ~ 10190 2395
+Wire Wire Line
+	9665 2995 10580 2995
 $Comp
 L R R4
 U 1 1 58AEAF1C
-P 4765 3745
-F 0 "R4" V 4845 3745 50  0000 C CNN
-F 1 "4.7k" V 4765 3745 50  0000 C CNN
-F 2 "Resistors_SMD:R_0805" V 4695 3745 50  0001 C CNN
-F 3 "" H 4765 3745 50  0001 C CNN
-	1    4765 3745
-	1    0    0    -1
-$EndComp
-Text GLabel 4765 3595 1    39   Input ~ 0
-3.3V
-Connection ~ 4765 3895
-Wire Wire Line
-	4390 3995 5640 3995
+P 10540 2845
+F 0 "R4" V 10620 2845 50  0000 C CNN
+F 1 "4.7k" V 10540 2845 50  0000 C CNN
+F 2 "Resistors_SMD:R_0805" V 10470 2845 50  0001 C CNN
+F 3 "" H 10540 2845 50  0001 C CNN
+	1    10540 2845
+	-1   0    0    -1
+$EndComp
+Text GLabel 10540 2695 1    39   Input ~ 0
+3.3V
+Connection ~ 10540 2995
+Wire Wire Line
+	9665 2895 10915 2895
 $Comp
 L R R3
 U 1 1 58AEB4D6
-P 4430 3845
-F 0 "R3" V 4510 3845 50  0000 C CNN
-F 1 "4.7k" V 4430 3845 50  0000 C CNN
-F 2 "Resistors_SMD:R_0805" V 4360 3845 50  0001 C CNN
-F 3 "" H 4430 3845 50  0001 C CNN
-	1    4430 3845
-	-1   0    0    1
-$EndComp
-Text GLabel 4430 3695 1    39   Input ~ 0
-3.3V
-Connection ~ 4430 3995
+P 10875 2745
+F 0 "R3" V 10955 2745 50  0000 C CNN
+F 1 "4.7k" V 10875 2745 50  0000 C CNN
+F 2 "Resistors_SMD:R_0805" V 10805 2745 50  0001 C CNN
+F 3 "" H 10875 2745 50  0001 C CNN
+	1    10875 2745
+	1    0    0    1
+$EndComp
+Text GLabel 10875 2595 1    39   Input ~ 0
+3.3V
+Connection ~ 10875 2895
 Text GLabel 8755 4875 0    39   Input ~ 0
 3.3V
@@
 NoConn ~ 7265 5470
 NoConn ~ 7265 5570
+$Comp
+L INA827 U1
+U 1 1 58AF6C20
+P 1505 2980
+F 0 "U1" H 1655 3105 50  0000 L CNN
+F 1 "INA827" H 1655 2855 50  0000 L CNN
+F 2 "Housings_SSOP:MSOP-8_3x3mm_Pitch0.65mm" H 1655 2780 50  0001 L CNN
+F 3 "" H 1605 2980 50  0001 C CNN
+	1    1505 2980
+	1    0    0    -1
+$EndComp
 $EndSCHEMATC
