File: SeniorDesignProject/SeniorDesign.sch (KiCad schematic (older format))
At the start: 27 parts, among them J1 RJ45(LoadCells), J2 RJ45(Accelerometer), J3 PICkit3, J4 RJ11(ICD3), J5 ID-12LA Header, J6 XBEE Header, J7 7-Segment Display, P7 Power 1, P9 Power 2, U1 INA827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

Commit message: Updates to board
Parts:
- removed J5: ID-12LA Header, Pin_Headers:Pin_Header_Straight_2x06_Pitch2.54mm, symbol CONN_02X06
- added J5: ID-12LA Header, Socket_Strips:Socket_Strip_Straight_1x05_Pitch2.54mm, symbol CONN_01X05
- added U2: LM1117-3.3, TO_SOT_Packages_SMD:SOT-223, symbol LM1117-3.3
Connections:
- net +5V: now also U9.VO, J5.1 (P1), U2.3 (VI)
- net -5V: now also U10.VO
- net 3.3V: now also U2.2 (VO), U2.4 (VO)
- net GND: now also P7.1 (P1), P9.2 (P2), U10.GND, U9.GND, J5.2 (P2), U2.1 (GND/ADJ)
- net SCL1: now also CPU1.37 (SCL1/RPI53/RC5), R6.2; no longer CPU1.48 (TCK/CVREF1O/ASCL1/RP40/T4CK/RB8), R5.2
- net SCL2: now also CPU1.32 (FLT32/SCL2/RP36/RB4); no longer CPU1.44 (PGEC2/ASCL2/RP38/RB6)
- net SDA1: now also CPU1.36 (SDA1/RPI52/RC4), R5.2; no longer CPU1.49 (TMS/ASDA1/RP41/RB9), R6.2
- net SDA2: now also CPU1.31 (SDA2/RPI24/RA8); no longer CPU1.43 (PGED2/ASDA2/RP37/RB5)
- net UART1RX: now also CPU1.51 (RP55/RC7), J5.4 (P4); no longer CPU1.45 (RPI58/RC10)
- net UART1TX: now also CPU1.50 (RP54/RC6); no longer CPU1.46 (RP39/INT0/RB7)
- net at P7.2 (P2): now also U9.VI
- net at U10.VI: now also P9.1 (P1)
- net AN0 renamed AN13
- new net CP: J5.5 (P5)
- new net LED: J5.3 (P3)
- no-connect marks 32 -> 26
Other:
- moved on the sheet: J6, P9, R3, R4, R5, R6, U10, U9

Commit message: Updates
Parts:
- U10, U9: footprint TO_SOT_Packages_THT:TO-220_Horizontal -> TO_SOT_Packages_THT:TO-92_Inline_Wide
Connections:
- net UART1RX: now also CPU1.46 (RP39/INT0/RB7); no longer CPU1.51 (RP55/RC7)
- net +9V: now reaches P7.2 (P2), U9.VI
- net -9V: now reaches P9.1 (P1), U10.VI
Other:
- moved on the sheet: U10, U9
Changed lines of the file:
@@
 L 7805 U9
 U 1 1 58461699
-P 1320 795
-F 0 "U9" H 1470 599 50  0000 C CNN
-F 1 "7805" H 1320 995 50  0000 C CNN
-F 2 "TO_SOT_Packages_THT:TO-220_Horizontal" H 1320 795 50  0001 C CNN
-F 3 "http://www.ti.com/lit/ds/symlink/lm7805.pdf" H 1320 795 50  0001 C CNN
-	1    1320 795
+P 1620 785
+F 0 "U9" H 1770 589 50  0000 C CNN
+F 1 "7805" H 1620 985 50  0000 C CNN
+F 2 "TO_SOT_Packages_THT:TO-92_Inline_Wide" H 1620 785 50  0001 C CNN
+F 3 "http://www.ti.com/lit/ds/symlink/lm7805.pdf" H 1620 785 50  0001 C CNN
+	1    1620 785
 	1    0    0    -1
 $EndComp
@@
 L 7905 U10
 U 1 1 584617C8
-P 1475 1595
-F 0 "U10" H 1625 1400 50  0000 C CNN
-F 1 "7905" H 1475 1795 50  0000 C CNN
-F 2 "TO_SOT_Packages_THT:TO-220_Horizontal" H 1475 1595 50  0001 C CNN
-F 3 "http://www.ti.com/lit/ds/symlink/lm7905.pdf" H 1475 1595 50  0001 C CNN
-	1    1475 1595
+P 1655 1590
+F 0 "U10" H 1805 1395 50  0000 C CNN
+F 1 "7905" H 1655 1790 50  0000 C CNN
+F 2 "TO_SOT_Packages_THT:TO-92_Inline_Wide" H 1655 1590 50  0001 C CNN
+F 3 "http://www.ti.com/lit/ds/symlink/lm7905.pdf" H 1655 1590 50  0001 C CNN
+	1    1655 1590
 	1    0    0    -1
 $EndComp
@@
 Text GLabel 9665 1095 2    39   Input ~ 0
 UART2RX
-Text GLabel 9665 2195 2    39   Input ~ 0
+Text GLabel 9665 2695 2    39   Input ~ 0
 UART1RX
 Text GLabel 9665 2295 2    39   Input ~ 0
@@
 	1    0    0    -1
 $EndComp
-Text GLabel 1320 1045 3    39   Input ~ 0
-GND
-Text GLabel 1720 745  2    39   Input ~ 0
+Text GLabel 1620 1035 3    39   Input ~ 0
+GND
+Text GLabel 2020 735  2    39   Input ~ 0
 +5V
 $Comp
@@
 Wire Wire Line
 	920  1545 1075 1545
-Text GLabel 1475 1845 3    39   Input ~ 0
-GND
-Text GLabel 1875 1545 2    39   Input ~ 0
+Text GLabel 1655 1840 3    39   Input ~ 0
+GND
+Text GLabel 2055 1540 2    39   Input ~ 0
 -5V
 Text GLabel 2285 1095 0    39   Input ~ 0
@@
 Text GLabel 2900 7465 0    39   Input ~ 0
 CP
+Text GLabel 920  745  1    39   Input ~ 0
++9V
+Text GLabel 1220 735  1    39   Input ~ 0
++9V
+Text GLabel 1075 1545 1    39   Input ~ 0
+-9V
+Text GLabel 1255 1540 1    39   Input ~ 0
+-9V
 $EndSCHEMATC
