File: SeniorDesignProject/SeniorDesign.sch (KiCad schematic (older format))
At the start: 26 parts, among them J1 RJ45(LoadCells), J2 RJ45(Accelerometer), J3 PICkit3, J5 ID-12LA Header, J6 XBEE Header, J7 7-Segment Display, P7 Power 1, U1 INA827, U2 LM1117-3.3, U3 ICL7660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

Commit message: Updates (Final design)
Parts:
- added C11: .33uF, Capacitors_THT:CP_Radial_D5.0mm_P2.00mm, symbol C
- added C12: .1uF, Capacitors_THT:CP_Radial_D5.0mm_P2.00mm, symbol C
- added C13, C14: 10uF, Capacitors_Tantalum_SMD:CP_Tantalum_Case-T_EIA-3528-12_Hand, symbol C
- C8: footprint Capacitors_THT:CP_Radial_D5.0mm_P2.00mm -> Capacitors_Tantalum_SMD:CP_Tantalum_Case-T_EIA-3528-12_Hand
Connections:
- wire segments 42 -> 54
Changed lines of the file:
@@
 F 0 "C8" V 10090 1665 50  0000 L CNN
 F 1 "10uF" V 10170 1635 50  0000 L CNN
-F 2 "Capacitors_THT:CP_Radial_D5.0mm_P2.00mm" H 9998 1545 50  0001 C CNN
+F 2 "Capacitors_Tantalum_SMD:CP_Tantalum_Case-T_EIA-3528-12_Hand" H 9998 1545 50  0001 C CNN
 F 3 "" H 9960 1695 50  0001 C CNN
 	1    9960 1695
@@
 Text GLabel 1205 3180 0    39   Input ~ 0
 A-
-Connection ~ 935  2830
-Wire Wire Line
-	935  2830 1205 2880
-Wire Wire Line
-	5015 1580 5485 1580
-Wire Wire Line
-	5510 1905 5510 1795
-Wire Wire Line
-	5510 1795 5640 1795
-Wire Wire Line
-	5025 1905 5510 1905
-Wire Wire Line
-	5485 1580 5485 1695
-Wire Wire Line
-	5485 1695 5640 1695
-Wire Wire Line
-	5025 2585 5485 2585
-Wire Wire Line
-	5510 2905 5510 2795
-Wire Wire Line
-	5510 2795 5640 2795
-Wire Wire Line
-	5015 2905 5510 2905
-Wire Wire Line
-	5485 2585 5485 2695
-Wire Wire Line
-	5485 2695 5640 2695
-Wire Wire Line
-	5015 3205 5485 3205
-Wire Wire Line
-	5510 3505 5510 3395
-Wire Wire Line
-	5510 3395 5640 3395
-Wire Wire Line
-	5025 3505 5510 3505
-Wire Wire Line
-	5485 3205 5485 3295
-Wire Wire Line
-	5485 3295 5640 3295
-Wire Wire Line
-	9810 1695 9665 1695
-Wire Wire Line
-	10045 1375 9820 1570
-Wire Wire Line
-	9820 1570 9665 1595
-Connection ~ 5260 3205
-Wire Wire Line
-	5335 2605 5335 2585
-Connection ~ 5335 2585
-Wire Wire Line
-	5335 1605 5335 1580
-Connection ~ 5335 1580
-Wire Wire Line
-	9665 3195 10070 3195
-Wire Wire Line
-	9665 3495 10165 3495
-Connection ~ 9870 3195
-Connection ~ 9870 3495
-Wire Wire Line
-	5640 1495 5410 1495
-Wire Wire Line
-	5410 1495 5410 1365
-Wire Wire Line
-	5025 1365 5110 1365
-Connection ~ 9820 1570
-Connection ~ 5260 3505
-Connection ~ 5335 2905
-Connection ~ 5335 1905
-Wire Wire Line
-	9820 1570 10105 1570
-Wire Wire Line
-	10105 1570 10105 1560
-Wire Wire Line
-	1505 2530 1505 2680
-Connection ~ 1505 2570
-Wire Wire Line
-	1505 3280 1505 3340
-Wire Wire Line
-	935  3130 1205 3080
 Text GLabel 5470 6690 1    39   Input ~ 0
 GND
@@
 Text GLabel 9665 2295 2    39   Input ~ 0
 UART1TX
-Wire Wire Line
-	9665 3695 10880 3695
 $Comp
 L R R5
@@
 Text GLabel 10815 3395 1    39   Input ~ 0
 3.3V
-Connection ~ 10815 3695
-Wire Wire Line
-	9665 3595 10505 3590
-Wire Wire Line
-	10505 3590 10545 3590
 $Comp
 L R R6
@@
 Text GLabel 10505 3290 1    39   Input ~ 0
 3.3V
-Connection ~ 10505 3590
 Text GLabel 2800 5510 0    39   Input ~ 0
 3.3V
@@
 Text GLabel 920  845  3    39   Input ~ 0
 GND
-Text GLabel 2285 1095 0    39   Input ~ 0
-+5V
-Text GLabel 2585 1395 3    39   Input ~ 0
-GND
-Text GLabel 2885 1095 2    39   Input ~ 0
+Text GLabel 2110 1090 0    39   Input ~ 0
++5V
+Text GLabel 2585 1430 3    39   Input ~ 0
+GND
+Text GLabel 3075 1100 2    39   Input ~ 0
 3.3V
 $Comp
@@
 Text GLabel 3210 1930 2    39   Input ~ 0
 -5V
-Text GLabel 1620 1035 3    39   Input ~ 0
+Text GLabel 1615 1105 3    39   Input ~ 0
 GND
 Text GLabel 2020 735  2    39   Input ~ 0
@@
 	1    0    0    -1
 $EndComp
-Wire Wire Line
-	3130 2530 3130 2430
-Wire Wire Line
-	3560 2020 3560 2145
 $Comp
 L C C10
@@
 Text GLabel 3560 2445 3    39   Input ~ 0
 GND
-Wire Wire Line
-	3130 1930 3130 2020
-Wire Wire Line
-	3130 2020 3560 2020
-Wire Wire Line
-	3210 1930 3130 1930
 Text GLabel 9665 2595 2    39   Input ~ 0
 LED
 Text GLabel 9665 2395 2    39   Input ~ 0
 CP
+$Comp
+L C C11
+U 1 1 58D2A716
+P 1220 885
+F 0 "C11" H 1245 985 50  0000 L CNN
+F 1 ".33uF" H 1245 785 50  0000 L CNN
+F 2 "Capacitors_THT:CP_Radial_D5.0mm_P2.00mm" H 1258 735 50  0001 C CNN
+F 3 "" H 1220 885 50  0001 C CNN
+	1    1220 885
+	1    0    0    -1
+$EndComp
+$Comp
+L C C12
+U 1 1 58D2AB02
+P 2020 885
+F 0 "C12" H 2045 985 50  0000 L CNN
+F 1 ".1uF" H 2045 785 50  0000 L CNN
+F 2 "Capacitors_THT:CP_Radial_D5.0mm_P2.00mm" H 2058 735 50  0001 C CNN
+F 3 "" H 2020 885 50  0001 C CNN
+	1    2020 885
+	1    0    0    -1
+$EndComp
+Connection ~ 935  2830
+Wire Wire Line
+	935  2830 1205 2880
+Wire Wire Line
+	5015 1580 5485 1580
+Wire Wire Line
+	5510 1905 5510 1795
+Wire Wire Line
+	5510 1795 5640 1795
+Wire Wire Line
+	5025 1905 5510 1905
+Wire Wire Line
+	5485 1580 5485 1695
+Wire Wire Line
+	5485 1695 5640 1695
+Wire Wire Line
+	5025 2585 5485 2585
+Wire Wire Line
+	5510 2905 5510 2795
+Wire Wire Line
+	5510 2795 5640 2795
+Wire Wire Line
+	5015 2905 5510 2905
+Wire Wire Line
+	5485 2585 5485 2695
+Wire Wire Line
+	5485 2695 5640 2695
+Wire Wire Line
+	5015 3205 5485 3205
+Wire Wire Line
+	5510 3505 5510 3395
+Wire Wire Line
+	5510 3395 5640 3395
+Wire Wire Line
+	5025 3505 5510 3505
+Wire Wire Line
+	5485 3205 5485 3295
+Wire Wire Line
+	5485 3295 5640 3295
+Wire Wire Line
+	9810 1695 9665 1695
+Wire Wire Line
+	10045 1375 9820 1570
+Wire Wire Line
+	9820 1570 9665 1595
+Connection ~ 5260 3205
+Wire Wire Line
+	5335 2605 5335 2585
+Connection ~ 5335 2585
+Wire Wire Line
+	5335 1605 5335 1580
+Connection ~ 5335 1580
+Wire Wire Line
+	9665 3195 10070 3195
+Wire Wire Line
+	9665 3495 10165 3495
+Connection ~ 9870 3195
+Connection ~ 9870 3495
+Wire Wire Line
+	5640 1495 5410 1495
+Wire Wire Line
+	5410 1495 5410 1365
+Wire Wire Line
+	5025 1365 5110 1365
+Connection ~ 9820 1570
+Connection ~ 5260 3505
+Connection ~ 5335 2905
+Connection ~ 5335 1905
+Wire Wire Line
+	9820 1570 10105 1570
+Wire Wire Line
+	10105 1570 10105 1560
+Wire Wire Line
+	1505 2530 1505 2680
+Connection ~ 1505 2570
+Wire Wire Line
+	1505 3280 1505 3340
+Wire Wire Line
+	935  3130 1205 3080
+Wire Wire Line
+	9665 3695 10880 3695
+Connection ~ 10815 3695
+Wire Wire Line
+	9665 3595 10505 3590
+Wire Wire Line
+	10505 3590 10545 3590
+Connection ~ 10505 3590
+Wire Wire Line
+	3130 2530 3130 2430
+Wire Wire Line
+	3560 2020 3560 2145
+Wire Wire Line
+	3130 1930 3130 2020
+Wire Wire Line
+	3130 2020 3560 2020
+Wire Wire Line
+	3210 1930 3130 1930
+Wire Wire Line
+	1220 1035 2020 1035
+Wire Wire Line
+	1615 1105 1620 1105
+Wire Wire Line
+	1620 1105 1620 1035
+Connection ~ 1620 1035
+$Comp
+L C C14
+U 1 1 58D2B7FA
+P 2945 1250
+F 0 "C14" H 2970 1350 50  0000 L CNN
+F 1 "10uF" H 2970 1150 50  0000 L CNN
+F 2 "Capacitors_Tantalum_SMD:CP_Tantalum_Case-T_EIA-3528-12_Hand" H 2983 1100 50  0001 C CNN
+F 3 "" H 2945 1250 50  0001 C CNN
+	1    2945 1250
+	1    0    0    -1
+$EndComp
+$Comp
+L C C13
+U 1 1 58D2BB13
+P 2225 1245
+F 0 "C13" H 2250 1345 50  0000 L CNN
+F 1 "10uF" H 2250 1145 50  0000 L CNN
+F 2 "Capacitors_Tantalum_SMD:CP_Tantalum_Case-T_EIA-3528-12_Hand" H 2263 1095 50  0001 C CNN
+F 3 "" H 2225 1245 50  0001 C CNN
+	1    2225 1245
+	1    0    0    -1
+$EndComp
+Wire Wire Line
+	2885 1095 3075 1095
+Wire Wire Line
+	2945 1095 2945 1100
+Wire Wire Line
+	3075 1095 3075 1100
+Connection ~ 2945 1095
+Wire Wire Line
+	2110 1095 2285 1095
+Wire Wire Line
+	2110 1095 2110 1090
+Connection ~ 2225 1095
+Wire Wire Line
+	2225 1400 2945 1400
+Wire Wire Line
+	2585 1400 2585 1395
+Wire Wire Line
+	2225 1400 2225 1395
+Connection ~ 2585 1400
+Wire Wire Line
+	2585 1430 2585 1405
 $EndSCHEMATC

Commit message: Version 2 updates 3.3V regulator with GND, 5V regulator with GND, and added via
Parts:
- removed U9: 7805, TO_SOT_Packages_THT:TO-92_Inline_Wide, symbol 7805
- added U4: 7805, TO_SOT_Packages_THT:TO-92_Inline_Wide, symbol 7805
Connections:
- wire segments 54 -> 67
Changed lines of the file:
@@
 Text GLabel 3210 1930 2    39   Input ~ 0
 -5V
-Text GLabel 1615 1105 3    39   Input ~ 0
+Text GLabel 1620 1075 3    39   Input ~ 0
 GND
-Text GLabel 2020 735  2    39   Input ~ 0
+Text GLabel 2020 730  2    39   Input ~ 0
 +5V
-Text GLabel 1220 735  1    39   Input ~ 0
+Text GLabel 1220 730  1    39   Input ~ 0
 +9V
-$Comp
-L 7805 U9
-U 1 1 58461699
-P 1620 785
-F 0 "U9" H 1770 589 50  0000 C CNN
-F 1 "7805" H 1620 985 50  0000 C CNN
-F 2 "TO_SOT_Packages_THT:TO-92_Inline_Wide" H 1620 785 50  0001 C CNN
-F 3 "http://www.ti.com/lit/ds/symlink/lm7805.pdf" H 1620 785 50  0001 C CNN
-	1    1620 785
-	1    0    0    -1
-$EndComp
 Text GLabel 5640 2295 0    39   Input ~ 0
 SS
@@
 L C C11
 U 1 1 58D2A716
-P 1220 885
-F 0 "C11" H 1245 985 50  0000 L CNN
-F 1 ".33uF" H 1245 785 50  0000 L CNN
-F 2 "Capacitors_THT:CP_Radial_D5.0mm_P2.00mm" H 1258 735 50  0001 C CNN
-F 3 "" H 1220 885 50  0001 C CNN
-	1    1220 885
+P 1220 880
+F 0 "C11" H 1245 980 50  0000 L CNN
+F 1 ".33uF" H 1245 780 50  0000 L CNN
+F 2 "Capacitors_THT:CP_Radial_D5.0mm_P2.00mm" H 1258 730 50  0001 C CNN
+F 3 "" H 1220 880 50  0001 C CNN
+	1    1220 880
 	1    0    0    -1
 $EndComp
@@
 L C C12
 U 1 1 58D2AB02
-P 2020 885
-F 0 "C12" H 2045 985 50  0000 L CNN
-F 1 ".1uF" H 2045 785 50  0000 L CNN
-F 2 "Capacitors_THT:CP_Radial_D5.0mm_P2.00mm" H 2058 735 50  0001 C CNN
-F 3 "" H 2020 885 50  0001 C CNN
-	1    2020 885
-	1    0    0    -1
-$EndComp
-Connection ~ 935  2830
-Wire Wire Line
-	935  2830 1205 2880
-Wire Wire Line
-	5015 1580 5485 1580
-Wire Wire Line
-	5510 1905 5510 1795
-Wire Wire Line
-	5510 1795 5640 1795
-Wire Wire Line
-	5025 1905 5510 1905
-Wire Wire Line
-	5485 1580 5485 1695
-Wire Wire Line
-	5485 1695 5640 1695
-Wire Wire Line
-	5025 2585 5485 2585
-Wire Wire Line
-	5510 2905 5510 2795
-Wire Wire Line
-	5510 2795 5640 2795
-Wire Wire Line
-	5015 2905 5510 2905
-Wire Wire Line
-	5485 2585 5485 2695
-Wire Wire Line
-	5485 2695 5640 2695
-Wire Wire Line
-	5015 3205 5485 3205
-Wire Wire Line
-	5510 3505 5510 3395
-Wire Wire Line
-	5510 3395 5640 3395
-Wire Wire Line
-	5025 3505 5510 3505
-Wire Wire Line
-	5485 3205 5485 3295
-Wire Wire Line
-	5485 3295 5640 3295
-Wire Wire Line
-	9810 1695 9665 1695
-Wire Wire Line
-	10045 1375 9820 1570
-Wire Wire Line
-	9820 1570 9665 1595
-Connection ~ 5260 3205
-Wire Wire Line
-	5335 2605 5335 2585
-Connection ~ 5335 2585
-Wire Wire Line
-	5335 1605 5335 1580
-Connection ~ 5335 1580
-Wire Wire Line
-	9665 3195 10070 3195
-Wire Wire Line
-	9665 3495 10165 3495
-Connection ~ 9870 3195
-Connection ~ 9870 3495
-Wire Wire Line
-	5640 1495 5410 1495
-Wire Wire Line
-	5410 1495 5410 1365
-Wire Wire Line
-	5025 1365 5110 1365
-Connection ~ 9820 1570
-Connection ~ 5260 3505
-Connection ~ 5335 2905
-Connection ~ 5335 1905
-Wire Wire Line
-	9820 1570 10105 1570
-Wire Wire Line
-	10105 1570 10105 1560
-Wire Wire Line
-	1505 2530 1505 2680
-Connection ~ 1505 2570
-Wire Wire Line
-	1505 3280 1505 3340
-Wire Wire Line
-	935  3130 1205 3080
-Wire Wire Line
-	9665 3695 10880 3695
-Connection ~ 10815 3695
-Wire Wire Line
-	9665 3595 10505 3590
-Wire Wire Line
-	10505 3590 10545 3590
-Connection ~ 10505 3590
-Wire Wire Line
-	3130 2530 3130 2430
-Wire Wire Line
-	3560 2020 3560 2145
-Wire Wire Line
-	3130 1930 3130 2020
-Wire Wire Line
-	3130 2020 3560 2020
-Wire Wire Line
-	3210 1930 3130 1930
-Wire Wire Line
-	1220 1035 2020 1035
-Wire Wire Line
-	1615 1105 1620 1105
-Wire Wire Line
-	1620 1105 1620 1035
-Connection ~ 1620 1035
+P 2020 880
+F 0 "C12" H 2045 980 50  0000 L CNN
+F 1 ".1uF" H 2045 780 50  0000 L CNN
+F 2 "Capacitors_THT:CP_Radial_D5.0mm_P2.00mm" H 2058 730 50  0001 C CNN
+F 3 "" H 2020 880 50  0001 C CNN
+	1    2020 880
+	1    0    0    -1
+$EndComp
 $Comp
 L C C14
@@
 	1    0    0    -1
 $EndComp
-Wire Wire Line
-	2885 1095 3075 1095
+Connection ~ 935  2830
+Wire Wire Line
+	935  2830 1205 2880
+Wire Wire Line
+	5015 1580 5335 1580
+Wire Wire Line
+	5335 1580 5485 1580
+Wire Wire Line
+	5510 1905 5510 1795
+Wire Wire Line
+	5510 1795 5640 1795
+Wire Wire Line
+	5025 1905 5335 1905
+Wire Wire Line
+	5335 1905 5510 1905
+Wire Wire Line
+	5485 1580 5485 1695
+Wire Wire Line
+	5485 1695 5640 1695
+Wire Wire Line
+	5025 2585 5335 2585
+Wire Wire Line
+	5335 2585 5485 2585
+Wire Wire Line
+	5510 2905 5510 2795
+Wire Wire Line
+	5510 2795 5640 2795
+Wire Wire Line
+	5015 2905 5335 2905
+Wire Wire Line
+	5335 2905 5510 2905
+Wire Wire Line
+	5485 2585 5485 2695
+Wire Wire Line
+	5485 2695 5640 2695
+Wire Wire Line
+	5015 3205 5260 3205
+Wire Wire Line
+	5260 3205 5485 3205
+Wire Wire Line
+	5510 3505 5510 3395
+Wire Wire Line
+	5510 3395 5640 3395
+Wire Wire Line
+	5025 3505 5260 3505
+Wire Wire Line
+	5260 3505 5510 3505
+Wire Wire Line
+	5485 3205 5485 3295
+Wire Wire Line
+	5485 3295 5640 3295
+Wire Wire Line
+	9810 1695 9665 1695
+Wire Wire Line
+	10045 1375 9820 1570
+Wire Wire Line
+	9820 1570 9665 1595
+Connection ~ 5260 3205
+Wire Wire Line
+	5335 2605 5335 2585
+Connection ~ 5335 2585
+Wire Wire Line
+	5335 1605 5335 1580
+Connection ~ 5335 1580
+Wire Wire Line
+	9665 3195 9870 3195
+Wire Wire Line
+	9870 3195 10070 3195
+Wire Wire Line
+	9665 3495 9870 3495
+Wire Wire Line
+	9870 3495 10165 3495
+Connection ~ 9870 3195
+Connection ~ 9870 3495
+Wire Wire Line
+	5640 1495 5410 1495
+Wire Wire Line
+	5410 1495 5410 1365
+Wire Wire Line
+	5025 1365 5110 1365
+Connection ~ 9820 1570
+Connection ~ 5260 3505
+Connection ~ 5335 2905
+Connection ~ 5335 1905
+Wire Wire Line
+	9820 1570 10105 1570
+Wire Wire Line
+	10105 1570 10105 1560
+Wire Wire Line
+	1505 2530 1505 2570
+Wire Wire Line
+	1505 2570 1505 2680
+Connection ~ 1505 2570
+Wire Wire Line
+	1505 3280 1505 3340
+Wire Wire Line
+	935  3130 1205 3080
+Wire Wire Line
+	9665 3695 10815 3695
+Wire Wire Line
+	10815 3695 10880 3695
+Connection ~ 10815 3695
+Wire Wire Line
+	9665 3595 10505 3590
+Wire Wire Line
+	10505 3590 10545 3590
+Connection ~ 10505 3590
+Wire Wire Line
+	3130 2530 3130 2430
+Wire Wire Line
+	3560 2020 3560 2145
+Wire Wire Line
+	3130 1930 3130 2020
+Wire Wire Line
+	3130 2020 3560 2020
+Wire Wire Line
+	3210 1930 3130 1930
+Wire Wire Line
+	2885 1095 2945 1095
+Wire Wire Line
+	2945 1095 3075 1095
 Wire Wire Line
 	2945 1095 2945 1100
@@
 Connection ~ 2945 1095
 Wire Wire Line
-	2110 1095 2285 1095
+	2110 1095 2225 1095
+Wire Wire Line
+	2225 1095 2285 1095
 Wire Wire Line
 	2110 1095 2110 1090
 Connection ~ 2225 1095
 Wire Wire Line
-	2225 1400 2945 1400
+	2225 1400 2585 1400
+Wire Wire Line
+	2585 1400 2945 1400
 Wire Wire Line
 	2585 1400 2585 1395
@@
 Wire Wire Line
 	2585 1430 2585 1405
+$Comp
+L 7805 U4
+U 1 1 58EA93CB
+P 1620 780
+F 0 "U4" H 1770 584 50  0000 C CNN
+F 1 "7805" H 1620 980 50  0000 C CNN
+F 2 "TO_SOT_Packages_THT:TO-92_Inline_Wide" H 1620 780 50  0001 C CNN
+F 3 "" H 1620 780 50  0001 C CNN
+	1    1620 780
+	1    0    0    -1
+$EndComp
+Wire Wire Line
+	1220 1030 1620 1030
+Wire Wire Line
+	1620 1030 2020 1030
+Connection ~ 1620 1030
+Wire Wire Line
+	1620 1075 1620 1030
 $EndSCHEMATC

Commit message: Updates to board
Other:
- moved on the sheet: C13, C14
Changed lines of the file:
@@
 L LM1117-3.3 U2
 U 1 1 58B786AE
-P 2585 1095
-F 0 "U2" H 2685 845 50  0000 C CNN
-F 1 "LM1117-3.3" H 2585 1345 50  0000 C CNN
-F 2 "TO_SOT_Packages_SMD:SOT-223" H 2585 1095 50  0001 C CNN
-F 3 "" H 2585 1095 50  0001 C CNN
-	1    2585 1095
+P 3325 850
+F 0 "U2" H 3425 600 50  0000 C CNN
+F 1 "LM1117-3.3" H 3325 1100 50  0000 C CNN
+F 2 "TO_SOT_Packages_SMD:SOT-223" H 3325 850 50  0001 C CNN
+F 3 "" H 3325 850 50  0001 C CNN
+	1    3325 850
 	1    0    0    -1
 $EndComp
 Text GLabel 920  845  3    39   Input ~ 0
 GND
-Text GLabel 2110 1090 0    39   Input ~ 0
+Text GLabel 2850 845  0    39   Input ~ 0
 +5V
-Text GLabel 2585 1430 3    39   Input ~ 0
-GND
-Text GLabel 3075 1100 2    39   Input ~ 0
+Text GLabel 3325 1185 3    39   Input ~ 0
+GND
+Text GLabel 3815 855  2    39   Input ~ 0
 3.3V
 $Comp
@@
 L C C14
 U 1 1 58D2B7FA
-P 2945 1250
-F 0 "C14" H 2970 1350 50  0000 L CNN
-F 1 "10uF" H 2970 1150 50  0000 L CNN
-F 2 "Capacitors_Tantalum_SMD:CP_Tantalum_Case-T_EIA-3528-12_Hand" H 2983 1100 50  0001 C CNN
-F 3 "" H 2945 1250 50  0001 C CNN
-	1    2945 1250
+P 3685 1005
+F 0 "C14" H 3710 1105 50  0000 L CNN
+F 1 "10uF" H 3710 905 50  0000 L CNN
+F 2 "Capacitors_Tantalum_SMD:CP_Tantalum_Case-T_EIA-3528-12_Hand" H 3723 855 50  0001 C CNN
+F 3 "" H 3685 1005 50  0001 C CNN
+	1    3685 1005
 	1    0    0    -1
 $EndComp
@@
 L C C13
 U 1 1 58D2BB13
-P 2225 1245
-F 0 "C13" H 2250 1345 50  0000 L CNN
-F 1 "10uF" H 2250 1145 50  0000 L CNN
-F 2 "Capacitors_Tantalum_SMD:CP_Tantalum_Case-T_EIA-3528-12_Hand" H 2263 1095 50  0001 C CNN
-F 3 "" H 2225 1245 50  0001 C CNN
-	1    2225 1245
+P 2965 1000
+F 0 "C13" H 2990 1100 50  0000 L CNN
+F 1 "10uF" H 2990 900 50  0000 L CNN
+F 2 "Capacitors_Tantalum_SMD:CP_Tantalum_Case-T_EIA-3528-12_Hand" H 3003 850 50  0001 C CNN
+F 3 "" H 2965 1000 50  0001 C CNN
+	1    2965 1000
 	1    0    0    -1
 $EndComp
@@
 	3210 1930 3130 1930
 Wire Wire Line
-	2885 1095 2945 1095
-Wire Wire Line
-	2945 1095 3075 1095
-Wire Wire Line
-	2945 1095 2945 1100
-Wire Wire Line
-	3075 1095 3075 1100
-Connection ~ 2945 1095
-Wire Wire Line
-	2110 1095 2225 1095
-Wire Wire Line
-	2225 1095 2285 1095
-Wire Wire Line
-	2110 1095 2110 1090
-Connection ~ 2225 1095
-Wire Wire Line
-	2225 1400 2585 1400
-Wire Wire Line
-	2585 1400 2945 1400
-Wire Wire Line
-	2585 1400 2585 1395
-Wire Wire Line
-	2225 1400 2225 1395
-Connection ~ 2585 1400
-Wire Wire Line
-	2585 1430 2585 1405
+	3625 850  3685 850
+Wire Wire Line
+	3685 850  3815 850
+Wire Wire Line
+	3685 850  3685 855
+Wire Wire Line
+	3815 850  3815 855
+Connection ~ 3685 850
+Wire Wire Line
+	2850 850  2965 850
+Wire Wire Line
+	2965 850  3025 850
+Wire Wire Line
+	2850 850  2850 845
+Connection ~ 2965 850
+Wire Wire Line
+	2965 1155 3325 1155
+Wire Wire Line
+	3325 1155 3685 1155
+Wire Wire Line
+	3325 1155 3325 1150
+Wire Wire Line
+	2965 1155 2965 1150
+Connection ~ 3325 1155
+Wire Wire Line
+	3325 1185 3325 1160
 $Comp
 L 7805 U4
