File: SeniorDesignProject/_saved_SeniorDesign.sch (KiCad schematic (older format))
At the start: 26 parts, among them J1 RJ45(LoadCells), J2 RJ45(Accelerometer), J3 PICkit3, J5 ID-12LA Header, J6 XBEE Header, J7 7-Segment Display, P7 Power 1, U1 INA827, U2 LM1117-3.3, U3 ICL7660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

Commit message: Re routed traces added tantalum cap for vcap
Parts:
- C8: footprint Capacitors_THT:CP_Radial_D5.0mm_P2.00mm -> Capacitors_Tantalum_SMD:CP_Tantalum_Case-T_EIA-3528-12_Hand
Changed lines of the file:
@@
 F 0 "C8" V 10090 1665 50  0000 L CNN
 F 1 "10uF" V 10170 1635 50  0000 L CNN
-F 2 "Capacitors_THT:CP_Radial_D5.0mm_P2.00mm" H 9998 1545 50  0001 C CNN
+F 2 "Capacitors_Tantalum_SMD:CP_Tantalum_Case-T_EIA-3528-12_Hand" H 9998 1545 50  0001 C CNN
 F 3 "" H 9960 1695 50  0001 C CNN
 	1    9960 1695
